Commit message: iCubGazeboV3: Remove XSense IMU pose and use original Bosch RFE IMU pose

File: iCub/robots/iCubGazeboV3/model.urdf (robot description, URDF)
Before this commit: robot iCub, 48 links, 47 joints
Joints:
- joint imu_frame_fixed_joint: origin xyz=0.009500000190735 0.133444 0.009299999999999996 rpy=-1.5707963267948961 1.570796326794896 0 -> xyz=0.0034999999997785457 0.0054999999863750895 0.1013340000004441 rpy=-3.141592653589793 0 -1.570796326794897
